File: display.kicad_sch (KiCad schematic)
At the start: 28 parts, among them J10 FH34SRJ-24S-0.5SH_99_E2417KS0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, Q3 Si1308EDL, U14 TXU0104PWR, U15 SN74LXC1T45DCKR, U16 TCK107AF,LF

Commit message: Use a different LED with better forward voltage
Change the main MCU LED to a one with better forward voltage.
Parts:
- J10, U15: Height 1.1 -> (none)
- U14: Height 1.2 -> (none)
- renumbered D2 to D3, D3 to D4, D4 to D5
