File: host_mcu.kicad_sch (KiCad schematic)
At the start: 33 parts, among them J2 TC2050, U5 nRF5340-QKxx, U6 MX25R3235FM1IH0-TR, Y1 32M, Y2 32k768

Commit message: Use a different LED with better forward voltage
Change the main MCU LED to a one with better forward voltage.
Connections:
- net GND: now also U5.A25 (VSS), U5.B12 (VSS), U5.B26 (VSS), U5.G1 (VSS), U5.H2 (VSS), U5.J31 (VSS)
