File: radio_mcu.kicad_sch (KiCad schematic)
At the start: 33 parts, among them Q1 RV2C010UNT2L, U7 TCK107AF,LF, U8 NRF7001-QFAA-R, U9 BGS12WN6E6327, Y3 Crystal_GND24

Commit message: Use a different LED with better forward voltage
Change the main MCU LED to a one with better forward voltage.
Parts:
- ANT1: Height 0.6 -> (none)
- FL1, U8: Height 0.9 -> (none)
- L6: Manufacturer_Name KYOCERA AVX -> Murata Electronics; Manufacturer_Part_Number L02011R5BHSTR -> LQP03HQ1N5B02D; Mouser Part Number 581-L02011R5BHSTR -> 81-LQP03HQ1N5B02D; Mouser Price/Stock https://www.mouser.co.uk/ProductDetail/KYOCERA-AVX/L02011R5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 -> https://www.mouser.co.uk/en/ProductDetail/Murata-Electronic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
