File: sensors.kicad_sch (KiCad schematic)
At the start: 49 parts, among them J3 SM05B-GHS-TB, J4 Header, J5 BM02B-ACHSS-GAN-ETF, J6 SM04B-GHS-TB, J7 SM04B-GHS-TB, J8 SM06B-GHS-TB, J9 SM06B-GHS-TB, Q2 RUM001L02T2CL, U10 SGP41-D-R4, U11 PCA9306D, U12 SRV05-4, U13 BME690

Commit message: Use a different LED with better forward voltage
Change the main MCU LED to a one with better forward voltage.
Parts:
- D2: renamed from LED1; value SML-D12U1WT86 -> APHD1608LSURCK; footprint SML-D12U1WT86:LEDC1608X65N -> LED_SMD:LED_0603_1608Metric; symbol SML-D12U1WT86:SML-D12U1WT86 -> Device:LED; Height 0.65 -> (none); Manufacturer_Name ROHM Semiconductor -> Kingbright; Manufacturer_Part_Number SML-D12U1WT86 -> APHD1608LSURCK; Mouser Part Number 755-SML-D12U1WT86 -> 604-APHD1608LSURCK; Mouser Price/Stock https://www.mouser.co.uk/ProductDetail/ROHM-Semiconductor/S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 -> https://www.mouser.co.uk/en/ProductDetail/Kingbright/APHD16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
- LS1: Height 2.5 -> (none)
- R30: value 1.5k -> 50; Manufacturer_Part_Number RC0402FR-7D1K5L -> RC0402JR-0750RL; Mouser Part Number 603-RC0402FR-7D1K5L -> 603-RC0402JR-0750RL; Mouser Price/Stock https://www.mouser.co.uk/ProductDetail/YAGEO/RC0402FR-7D1K5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 -> https://www.mouser.co.uk/ProductDetail/YAGEO/RC0402JR-0750R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
- S1: Height 1.35 -> (none)
- U10: Height 0.95 -> (none)
- U13: Height 1 -> (none)
