File: sheets/host_mcu.kicad_sch (KiCad schematic)
At the start: 33 parts, among them J2 TC2050, U5 nRF5340-QKxx, U6 MX25R3235FM1IH0-TR, Y1 32M, Y2 32k768

Commit message: Add project symbols and footprints
Move all self-made symbols and footprints to the lib folder.
Parts:
- U5: footprint MyLib:Nordic_AQFN-94-1EP_7x7mm_P0.4mm -> nRF5340-QKxx:Nordic_AQFN-94-1EP_7x7mm_P0.4mm; symbol MCU_Nordic:nRF5340-QKxx -> nRF5340-QKxx:nRF5340-QKxx
Changed lines of the file:
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@@
 	)
 	(symbol
-		(lib_id "MCU_Nordic:nRF5340-QKxx")
+		(lib_id "nRF5340-QKxx:nRF5340-QKxx")
 		(at 115.57 107.95 0)
 		(unit 1)
@@
 			)
 		)
-		(property "Footprint" "MyLib:Nordic_AQFN-94-1EP_7x7mm_P0.4mm"
+		(property "Footprint" "nRF5340-QKxx:Nordic_AQFN-94-1EP_7x7mm_P0.4mm"
 			(at 151.13 34.29 0)
 			(hide yes)
