File: sheets/power.kicad_sch (KiCad schematic)
At the start: 34 parts, among them J1 USB_C_Receptacle_USB2.0_16P, U1 TLV70033DDCR, U2 TLV70036DDCR, U3 USBLC6-2SC6, U4 TPS2553DDBVR

Commit message: Add project symbols and footprints
Move all self-made symbols and footprints to the lib folder.
Parts:
- D1: footprint SMBJ5.0A:DIOM5436X244N -> Diode_SMD:D_SMB; symbol SMBJ5_0A:SMBJ5.0A -> Device:D_Zener
- F1: footprint MyLib:Fuse_SF-1206F -> Fuse:Fuse_1206_3216Metric
- U1: footprint TLV70033DDCR:SOT95P280X110-5N -> Package_TO_SOT_SMD:SOT-23-5; symbol TLV70033DDCR:TLV70033DDCR -> Regulator_Linear:TLV70033_SOT23-5
- U2: footprint TLV70036DDCR:SOT95P280X110-5N -> Package_TO_SOT_SMD:SOT-23-5; symbol TLV70036DDCR:TLV70036DDCR -> Regulator_Linear:TLV70036_SOT23-5
- U4: footprint TPS2553DDBVR:SOT95P280X145-6N -> Package_TO_SOT_SMD:SOT-23-6; symbol TPS2553DDBVR:TPS2553DDBVR -> TPS255xD:TPS2553D
Connections:
- net +Vbus: now also D1.1 (K); no longer D1.2 (A)
- net GND: now also D1.2 (A); no longer D1.1 (K)
- no-connect marks 4 -> 2
Other:
- moved on the sheet: C3, C4, C5, C7, R3, R4, R5, R6, R7, U4
