File: sheets/radio_mcu.kicad_sch (KiCad schematic)
At the start: 33 parts, among them Q1 RV2C010UNT2L, U7 TCK107AF,LF, U8 NRF7001-QFAA-R, U9 BGS12WN6E6327, Y3 Crystal_GND24

Commit message: Add project symbols and footprints
Move all self-made symbols and footprints to the lib folder.
Parts:
- AE1: renamed from ANT1; symbol 2450AD18A6050001E:2450AD18A6050001E -> Antenna:Antenna_NC
- Q1: footprint RV2C010UNT2L:RV2C010UNT2L -> RV2C010UNT2L-Small:RV2C010UNT2L
- U7: symbol TCK107AF_LF:TCK107AF,LF -> TCK10xAF:TCK107AF
- U8: footprint NRF7001-QFAA-R:QFN40P600X600X90-49N -> Package_DFN_QFN:QFN-48-1EP_6x6mm_P0.4mm_EP4.66x4.66mm; symbol NRF7001-QFAA-R:NRF7001-QFAA-R -> nRF7001:nRF7001
- U9: footprint MyLib:Infineon_PG-TSNP-6-10_0.7x1.1mm_0.7x1.1mm_P0.4mm -> BGS12WN6E6327:Infineon_PG-TSNP-6-10_0.7x1.1mm_0.7x1.1mm_P0.4mm
Connections:
- no-connect marks 13 -> 1
Other:
- moved on the sheet: C31, C32, C33, C34, C35, C36, C37, C38, C39, C40, C41, C42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
